File: hardware/HotPotato.brd (EAGLE design)
At the start: 38 x 27.3 mm, 15 parts, among them K1 TS-1101F, M1 SANYO_NRS-2574SMT, SW1 TACTILE-SWITCH-PTH, U1 TINY85-20-DIP

Commit message: Increase distance between buzzer poles
Fixes #4
Parts:
- removed SG2: BUZZER, dhgoldberg:BUZZER-9MM-PTH
- added SG1: BUZZER9MM, dhgoldberg:BUZZER-9MM-PTH_NEW
- D3: device SparkFun-LED:LED5MM-KIT -> SparkFun-LED:LED_5MM-KIT
- moved D3 0.50 mm to (96.3, 64.6), turned to 135 degrees
Connections:
- net BUZZ: now also SG1.P$1; no longer SG2.P$1
- net N$5: now also SG1.P$2; no longer SG2.P$2
Routing:
- net ACC_POW: track 23.1 -> 20.1 mm
- net ACC_IN: track 25.3 -> 22.7 mm
- net N$5: track 7.97 -> 5.65 mm
- net N$2: track 7.06 -> 5.76 mm
Other:
- board text added: "BUZZER"
- board text added: "rev. 2 designed by Dimitris Platis"
- board text removed: "rev. 1 designed by Dimitris Platis"
Changed lines of the file:
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@@
 <?xml version="1.0" encoding="utf-8"?>
 <!DOCTYPE eagle SYSTEM "eagle.dtd">
-<eagle version="8.1.1">
+<eagle version="8.3.0">
 <drawing>
 <settings>
 <setting alwaysvectorfont="no"/>
+<setting keepoldvectorfont="yes"/>
 <setting verticaltext="up"/>
 </settings>
@@
 <text x="72.65" y="42.9" size="0.8128" layer="21" font="vector">ACC_X</text>
 <text x="102.7" y="52.8" size="1.9304" layer="22" font="vector" rot="MR0">Scrumtato</text>
-<text x="95.8" y="48.3" size="1.016" layer="22" font="vector" rot="MR0" align="bottom-center">rev. 1
+<text x="95.8" y="48.3" size="1.016" layer="22" font="vector" rot="MR0" align="bottom-center">rev. 2
 designed by
 Dimitris Platis</text>
+<text x="74.25" y="50" size="0.8128" layer="21" font="vector" rot="R225">BUZZER</text>
 </plain>
 <attributes>
@@
 <attribute name="VALUE" x="82.32" y="58.25" size="0.8128" layer="27" ratio="10"/>
 </element>
-<element name="D3" library="SparkFun-LED" package="LED5MM-KIT" value="" x="96.845" y="64.58" smashed="yes" rot="R270">
-<attribute name="NAME" x="92.281" y="65.992" size="0.8128" layer="25"/>
-<attribute name="VALUE" x="95.067" y="65.596" size="0.4064" layer="27" rot="R270"/>
+<element name="D3" library="SparkFun-LED" library_urn="urn:adsk.eagle:library:529" package="LED_5MM-KIT" package3d_urn="urn:adsk.eagle:package:39357/1" value="" x="96.345" y="64.58" smashed="yes" rot="R135">
+<attribute name="NAME" x="93.32066875" y="66.808803125" size="0.8128" layer="25" rot="R225"/>
+<attribute name="VALUE" x="98.32065625" y="65.118815625" size="0.4064" layer="27" rot="R135"/>
 </element>
 <element name="M1" library="dhgoldberg" package="SMT" value="SANYO_NRS-2574SMT" x="100.58" y="54.57" smashed="yes" rot="R270"/>
@@
 <attribute name="VALUE" x="68.736975" y="59.366978125" size="0.4064" layer="27" ratio="10" rot="R270"/>
 </element>
-<element name="SG2" library="dhgoldberg" package="BUZZER-9MM-PTH" value="BUZZER" x="74.31" y="46.91" rot="R270"/>
-<element name="Q2" library="SparkFun-DiscreteSemi" package="TO-92-AMMO" value="" x="95.25" y="44.5" smashed="yes">
+<element name="Q2" library="SparkFun-DiscreteSemi" library_urn="urn:adsk.eagle:library:514" package="TO-92-AMMO" value="" x="95.25" y="44.5" smashed="yes">
 <attribute name="NAME" x="97.925" y="45.905" size="0.8128" layer="25" ratio="10"/>
 <attribute name="VALUE" x="98.425" y="42.595" size="0.4064" layer="27" ratio="10"/>
 </element>
-<element name="J1" library="SparkFun-Connectors" package="1X05" value="" x="72.15" y="41.2" smashed="yes">
+<element name="J1" library="SparkFun-Connectors" library_urn="urn:adsk.eagle:library:513" package="1X05" value="" x="72.15" y="41.2" smashed="yes">
 <attribute name="NAME" x="69.5538" y="40.2788" size="0.8128" layer="25" ratio="10"/>
 <attribute name="VALUE" x="70.88" y="38.025" size="1.27" layer="27"/>
@@
 <attribute name="VALUE" x="83.405" y="68.195" size="0.6096" layer="27" ratio="11" rot="R180"/>
 </element>
+<element name="SG1" library="dhgoldberg" package="BUZZER-9MM-PTH_NEW" value="BUZZER9MM" x="74" y="47" rot="R225"/>
 </elements>
 <signals>
@@
 <contactref element="D3" pad="A"/>
 <contactref element="R2" pad="2"/>
-<wire x1="101.805" y1="60.845" x2="101.805" y2="60.89" width="0.6096" layer="1"/>
-<wire x1="101.805" y1="60.89" x2="96.845" y2="65.85" width="0.6096" layer="1"/>
+<wire x1="101.805" y1="60.89" x2="101.805" y2="60.845" width="0.6096" layer="1"/>
+<wire x1="97.243025" y1="63.681971875" x2="99.013028125" y2="63.681971875" width="0.6096" layer="1"/>
+<wire x1="99.013028125" y1="63.681971875" x2="101.805" y2="60.89" width="0.6096" layer="1"/>
 </signal>
 <signal name="SW">
@@
 <signal name="N$5">
 <contactref element="R4" pad="2"/>
-<contactref element="SG2" pad="P$2"/>
-<wire x1="67.095" y1="46.74" x2="68.925" y2="44.91" width="0.6096" layer="1"/>
-<wire x1="68.925" y1="44.91" x2="74.31" y2="44.91" width="0.6096" layer="1"/>
+<contactref element="SG1" pad="P$2"/>
+<wire x1="72.04696875" y1="45.04696875" x2="68.78803125" y2="45.04696875" width="0.6096" layer="1"/>
+<wire x1="68.78803125" y1="45.04696875" x2="67.095" y2="46.74" width="0.6096" layer="1"/>
 </signal>
 <signal name="BUZZ">
-<contactref element="SG2" pad="P$1"/>
 <contactref element="U1" pad="5"/>
 <contactref element="R2" pad="1"/>
-<wire x1="74.681975" y1="52.631978125" x2="72.4" y2="54.913953125" width="0.6096" layer="1"/>
-<wire x1="74.31" y1="48.91" x2="74.681975" y2="49.281975" width="0.6096" layer="1"/>
-<wire x1="74.681975" y1="49.281975" x2="74.681975" y2="52.631978125" width="0.6096" layer="1"/>
+<wire x1="72.4" y1="54.913953125" x2="74.681975" y2="52.631978125" width="0.6096" layer="1"/>
 <wire x1="95.905" y1="60.845" x2="91" y2="65.75" width="0.6096" layer="1"/>
 <wire x1="95.905" y1="60.845" x2="99.005" y2="60.845" width="0.6096" layer="1"/>
@@
 <wire x1="72.4" y1="54.913953125" x2="72.4" y2="63.9" width="0.6096" layer="1"/>
 <wire x1="72.4" y1="63.9" x2="72.75" y2="64.25" width="0.6096" layer="1"/>
+<contactref element="SG1" pad="P$1"/>
+<wire x1="74.681975" y1="52.631978125" x2="74.681975" y2="50.22408125" width="0.6096" layer="1"/>
+<wire x1="74.681975" y1="50.22408125" x2="75.953028125" y2="48.953028125" width="0.6096" layer="1"/>
 </signal>
 <signal name="MOT">
@@
 <contactref element="U1" pad="3"/>
 <contactref element="J1" pad="1"/>
-<wire x1="69.5" y1="54.3" x2="69.5" y2="48.3" width="0.6096" layer="1"/>
+<wire x1="69.5" y1="54.3" x2="69.5" y2="47.5" width="0.6096" layer="1"/>
 <wire x1="67.061975" y1="55.171978125" x2="68.628021875" y2="55.171978125" width="0.6096" layer="1"/>
 <wire x1="68.628021875" y1="55.171978125" x2="69.5" y2="54.3" width="0.6096" layer="1"/>
-<wire x1="69.5" y1="48.3" x2="69.5" y2="47.5" width="0.6096" layer="1"/>
-<wire x1="69.5" y1="47.5" x2="70.75" y2="46.25" width="0.6096" layer="1"/>
-<wire x1="70.75" y1="46.25" x2="75.25" y2="46.25" width="0.6096" layer="1"/>
-<wire x1="75.25" y1="46.25" x2="76" y2="45.5" width="0.6096" layer="1"/>
-<wire x1="76" y1="45.5" x2="76" y2="44.5" width="0.6096" layer="1"/>
-<wire x1="74.75" y1="43.25" x2="74.2" y2="43.25" width="0.6096" layer="1"/>
-<wire x1="74.2" y1="43.25" x2="72.15" y2="41.2" width="0.6096" layer="1"/>
-<wire x1="76" y1="44.5" x2="74.75" y2="43.25" width="0.6096" layer="1"/>
+<wire x1="69.5" y1="47.5" x2="70.25" y2="46.75" width="0.6096" layer="1"/>
+<wire x1="70.25" y1="46.75" x2="73" y2="46.75" width="0.6096" layer="1"/>
+<wire x1="73" y1="46.75" x2="74" y2="45.75" width="0.6096" layer="1"/>
+<wire x1="74" y1="43.5" x2="72.15" y2="41.65" width="0.6096" layer="1"/>
+<wire x1="72.15" y1="41.65" x2="72.15" y2="41.2" width="0.6096" layer="1"/>
+<wire x1="74" y1="45.75" x2="74" y2="43.5" width="0.6096" layer="1"/>
 </signal>
 <signal name="N$3">
@@
 <wire x1="67.061975" y1="57.711978125" x2="69.038021875" y2="57.711978125" width="0.6096" layer="1"/>
 <wire x1="69.038021875" y1="57.711978125" x2="70.75" y2="56" width="0.6096" layer="1"/>
-<wire x1="74.69" y1="41.2" x2="76.5" y2="43.01" width="0.6096" layer="1"/>
-<wire x1="76.5" y1="43.01" x2="76.51" y2="43.01" width="0.6096" layer="1"/>
-<wire x1="77.25" y1="43.75" x2="76.51" y2="43.01" width="0.6096" layer="1"/>
-<wire x1="70.75" y1="49.25" x2="72.5" y2="47.5" width="0.6096" layer="1"/>
-<wire x1="72.5" y1="47.5" x2="76.5" y2="47.5" width="0.6096" layer="1"/>
-<wire x1="76.5" y1="47.5" x2="77.25" y2="46.75" width="0.6096" layer="1"/>
 <wire x1="70.75" y1="56" x2="70.75" y2="49.25" width="0.6096" layer="1"/>
-<wire x1="77.25" y1="46.75" x2="77.25" y2="43.75" width="0.6096" layer="1"/>
+<wire x1="70.75" y1="49.25" x2="71.75" y2="48.25" width="0.6096" layer="1"/>
+<wire x1="71.75" y1="48.25" x2="73.75" y2="48.25" width="0.6096" layer="1"/>
+<wire x1="73.75" y1="48.25" x2="75.5" y2="46.5" width="0.6096" layer="1"/>
+<wire x1="75.5" y1="46.5" x2="75.5" y2="42.01" width="0.6096" layer="1"/>
+<wire x1="75.5" y1="42.01" x2="74.69" y2="41.2" width="0.6096" layer="1"/>
 </signal>
 <signal name="N$6">
@@
 which will not be processed correctly with this version.
 </note>
+<note version="8.2" severity="warning">
+Since Version 8.2, EAGLE supports online libraries. The ids
+of those online libraries will not be understood (or retained)
+with this version.
+</note>
+<note version="8.3" severity="warning">
+Since Version 8.3, EAGLE supports URNs for individual library
+assets (packages, symbols, and devices). The URNs of those assets
+will not be understood (or retained) with this version.
+</note>
+<note version="8.3" severity="warning">
+Since Version 8.3, EAGLE supports the association of 3D packages
+with devices in libraries, schematics, and board files. Those 3D
+packages will not be understood (or retained) with this version.
+</note>
 </compatibility>

Commit message: Remove accelerometer header and set dedicated LED pin
[hw rev. 3]
Since the Hot Potato (game) use case was deemed less significant
hardware support for it was removed in order to leave more space
for the common components. This also enabled us to use a dedicated
pin for the LED which was previously routed in parallel with the
buzzer.  This should enable better control over the hardware and
(theoretically) more current to be supplied to the LED and the
buzzer.
Parts:
- removed J1: (no value), SparkFun-Connectors:1X05
- moved R3 2.64 mm to (80.8, 41.2)
- moved SG1 1.00 mm to (74.0, 46.0)
Connections:
- removed net ACC_IN: J1.2, U1.2
- removed net ACC_POW: J1.1, U1.3
- new net LED: R2.1, U1.2
- net BUZZ: no longer R2.1
- net GND: no longer J1.5
Routing:
- net BUZZ: track 45.8 -> 5.21 mm
- net LED: track 0.00 -> 39.6 mm
- net ACC_IN: track 22.7 -> 0.00 mm
- net ACC_POW: track 20.1 -> 0.00 mm
- net GND: track 7.03 -> 18.8 mm
- net N$1: track 14.9 -> 16.9 mm
- net VCC: track 65.9 -> 64.8 mm
Other:
- board text added: "rev. 3 designed by Dimitris Platis"
- board text removed: "ACC_X"
- board text removed: "GND"
- board text removed: "VCC"
- board text removed: "rev. 2 designed by Dimitris Platis"
